File: projects/UnoSensor/UnoSensor.sch (EAGLE design)
At the start: 8 parts

Commit message: init
Parts:
- removed LED1: (no value), adafruit:LEDCHIPLED_0603
- removed R1: 330, adafruit:R-US_M0805
Connections:
- removed net N$2: R1.2, U5.3V3
- removed net N$8: LED1.A, R1.1
- removed net N$9: LED1.C, U5.GND@1
Changed lines of the file:
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@@
 <part name="SV3" library="CON_LSTB" deviceset="MA03-1" device=""/>
 <part name="SV4" library="CON_LSTB" deviceset="MA03-1" device=""/>
-<part name="LED1" library="adafruit" deviceset="LED" device="CHIPLED_0603"/>
-<part name="R1" library="adafruit" deviceset="R-US_" device="M0805" value="330"/>
 <part name="SW1" library="SPECIAL" deviceset="SW_DIP-6" device=""/>
 </parts>
@@
 <attribute name="VALUE" x="-62.23" y="-66.04" size="1.778" layer="96"/>
 <attribute name="NAME" x="-62.23" y="-52.578" size="1.778" layer="95"/>
-</instance>
-<instance part="LED1" gate="G$1" x="-35.56" y="68.58" smashed="yes" rot="R270">
-<attribute name="NAME" x="-40.132" y="65.024" size="1.778" layer="95"/>
-<attribute name="VALUE" x="-40.132" y="62.865" size="1.778" layer="96"/>
-</instance>
-<instance part="R1" gate="G$1" x="-22.86" y="68.58" smashed="yes">
-<attribute name="NAME" x="-26.67" y="70.0786" size="1.778" layer="95"/>
-<attribute name="VALUE" x="-26.67" y="65.278" size="1.778" layer="96"/>
 </instance>
 <instance part="SW1" gate="A" x="-43.18" y="35.56" smashed="yes">
@@
 </segment>
 </net>
-<net name="N$2" class="0">
-<segment>
-<pinref part="U5" gate="SEEEDUINO" pin="3V3"/>
-<pinref part="R1" gate="G$1" pin="2"/>
-<wire x1="-10.16" y1="57.15" x2="-17.78" y2="57.15" width="0.1524" layer="91"/>
-<wire x1="-17.78" y1="57.15" x2="-17.78" y2="68.58" width="0.1524" layer="91"/>
-</segment>
-</net>
-<net name="N$8" class="0">
-<segment>
-<pinref part="R1" gate="G$1" pin="1"/>
-<pinref part="LED1" gate="G$1" pin="A"/>
-<wire x1="-27.94" y1="68.58" x2="-33.02" y2="68.58" width="0.1524" layer="91"/>
-</segment>
-</net>
-<net name="N$9" class="0">
-<segment>
-<pinref part="LED1" gate="G$1" pin="C"/>
-<wire x1="-40.64" y1="68.58" x2="-43.18" y2="68.58" width="0.1524" layer="91"/>
-<wire x1="-43.18" y1="68.58" x2="-43.18" y2="48.26" width="0.1524" layer="91"/>
-<pinref part="U5" gate="SEEEDUINO" pin="GND@1"/>
-<wire x1="-43.18" y1="48.26" x2="-10.16" y2="48.26" width="0.1524" layer="91"/>
-<wire x1="-10.16" y1="48.26" x2="-10.16" y2="49.53" width="0.1524" layer="91"/>
-</segment>
-</net>
