File: projects/RpiStack/RpiStack.brd (EAGLE design)
At the start: 65 x 56.5 mm, 13 parts, among them T1 AP2302GN-HF/SOT23

Commit message: init
Parts:
- moved LORA_ANT 1.35 mm to (14.4, 2.83)
Routing:
- net ANT: track 6.09 -> 7.44 mm
Changed lines of the file:
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@@
 <drawing>
 <settings>
-<setting alwaysvectorfont="no"/>
+<setting alwaysvectorfont="yes"/>
 <setting keepoldvectorfont="yes"/>
 <setting verticaltext="up"/>
@@
 <attribute name="VALUE" x="13.395959375" y="32.98951875" size="0.8128" layer="27" rot="R270"/>
 </element>
-<element name="LORA_ANT" library="sma-ke" package="SMA-KE" value="SMA-KE" x="14.411959375" y="4.175759375" smashed="yes">
-<attribute name="NAME" x="18.503759375" y="3.555159375" size="1.27" layer="25" font="vector"/>
-<attribute name="VALUE" x="15.681959375" y="7.985759375" size="0.8128" layer="27"/>
+<element name="LORA_ANT" library="sma-ke" package="SMA-KE" value="SMA-KE" x="14.373859375" y="2.829559375" smashed="yes">
+<attribute name="NAME" x="18.465659375" y="2.208959375" size="1.27" layer="25" font="vector"/>
+<attribute name="VALUE" x="15.643859375" y="6.639559375" size="0.8128" layer="27"/>
 </element>
 <element name="U$2" library="lorarpi" package="RPILORASHIELD" value="RPILORASHIELD" x="32.826959375" y="28.41751875" smashed="yes"/>
@@
 <via x="9.738359375" y="2.86511875" extent="1-16" drill="0.3302" diameter="0.9652"/>
 <via x="15.224759375" y="53.268878125" extent="1-16" drill="0.3302" diameter="0.9652"/>
-<via x="15.097759375" y="55.36691875" extent="1-16" drill="0.3302" diameter="0.9652"/>
+<via x="15.097759375" y="55.32881875" extent="1-16" drill="0.3302" diameter="0.9652"/>
 <via x="25.079959375" y="55.26531875" extent="1-16" drill="0.3302" diameter="0.9652"/>
 <via x="43.012359375" y="52.97931875" extent="1-16" drill="0.3302" diameter="0.9652"/>
@@
 <wire x1="15.046959375" y1="53.091078125" x2="15.046959375" y2="52.91751875" width="0" layer="19" extent="1-1"/>
 <wire x1="12.506959375" y1="55.34151875" x2="13.806959375" y2="54.15751875" width="0" layer="19" extent="1-1"/>
-<wire x1="15.097759375" y1="55.36691875" x2="13.806959375" y2="54.15751875" width="0" layer="19" extent="1-1"/>
+<wire x1="15.097759375" y1="55.32881875" x2="13.806959375" y2="54.15751875" width="0" layer="19" extent="1-1"/>
 <wire x1="23.555959375" y1="31.46551875" x2="22.920959375" y2="36.03751875" width="0" layer="19" extent="1-1"/>
 <wire x1="6.537959375" y1="45.56251875" x2="11.236959375" y2="43.78451875" width="0" layer="19" extent="1-1"/>
@@
 <wire x1="22.413959375" y1="7.30631875" x2="18.856959375" y2="7.20851875" width="0" layer="19" extent="1-1"/>
 <wire x1="23.428959375" y1="4.79551875" x2="22.413959375" y2="7.30631875" width="0" layer="19" extent="1-1"/>
-<wire x1="17.011959375" y1="4.175759375" x2="18.856959375" y2="7.20851875" width="0" layer="19" extent="16-16"/>
-<wire x1="17.011959375" y1="4.175759375" x2="17.011959375" y2="4.175759375" width="0" layer="19" extent="1-16"/>
-<wire x1="11.811959375" y1="4.175759375" x2="17.011959375" y2="4.175759375" width="0" layer="19" extent="1-16"/>
-<wire x1="11.811959375" y1="4.175759375" x2="11.811959375" y2="4.175759375" width="0" layer="19" extent="1-16"/>
-<wire x1="9.738359375" y1="2.86511875" x2="11.811959375" y2="4.175759375" width="0" layer="19" extent="1-1"/>
-<wire x1="11.236959375" y1="8.85951875" x2="11.811959375" y2="4.175759375" width="0" layer="19" extent="1-1"/>
+<wire x1="16.973859375" y1="2.829559375" x2="18.856959375" y2="7.20851875" width="0" layer="19" extent="16-16"/>
+<wire x1="16.973859375" y1="2.829559375" x2="16.973859375" y2="2.829559375" width="0" layer="19" extent="1-16"/>
+<wire x1="11.773859375" y1="2.829559375" x2="16.973859375" y2="2.829559375" width="0" layer="19" extent="1-16"/>
+<wire x1="11.773859375" y1="2.829559375" x2="11.773859375" y2="2.829559375" width="0" layer="19" extent="1-16"/>
+<wire x1="9.738359375" y1="2.86511875" x2="11.773859375" y2="2.829559375" width="0" layer="19" extent="1-1"/>
+<wire x1="11.236959375" y1="8.85951875" x2="11.773859375" y2="2.829559375" width="0" layer="19" extent="1-1"/>
 <wire x1="56.327040625" y1="46.131478125" x2="55.661559375" y2="52.95391875" width="0" layer="19" extent="1-1"/>
 <wire x1="45.755559375" y1="12.77111875" x2="43.7032375" y2="19.3700375" width="0" layer="19" extent="1-1"/>
@@
 <contactref element="LORA" pad="9"/>
 <contactref element="LORA_ANT" pad="P$5"/>
-<wire x1="14.396959375" y1="10.25751875" x2="14.396959375" y2="4.190759375" width="1" layer="1"/>
-<wire x1="14.396959375" y1="4.190759375" x2="14.411959375" y2="4.175759375" width="1" layer="1"/>
+<wire x1="14.396959375" y1="10.25751875" x2="14.396959375" y2="2.852659375" width="1" layer="1"/>
+<wire x1="14.396959375" y1="2.852659375" x2="14.373859375" y2="2.829559375" width="1" layer="1"/>
 </signal>
 <signal name="RESET">
